File: IOSEC8.brd (EAGLE design)
At the start: 133.3 x 48.3 mm, 27 parts

Commit message: Moved to metric grid for v2.0 release
Parts:
- moved LED2 14.0 mm to (84.6, 5.35)
- moved R2 10.2 mm to (89.4, 5.35), turned to 180 degrees
- moved JP1 5.59 mm to (60.9, 3.85)
- moved J1 5.00 mm to (3.66, 22.9)
- moved J2 5.00 mm to (20.2, 22.9)
- moved J3 5.00 mm to (36.7, 22.9)
- moved J4 5.00 mm to (53.2, 22.9)
- moved J5 5.00 mm to (69.7, 22.9)
- moved J6 5.00 mm to (86.2, 22.9)
- moved J7 5.00 mm to (102.7, 22.9)
- moved J8 5.00 mm to (119.2, 22.9)
- moved R10 5.00 mm to (43.2, 16.6)
- moved R11 5.00 mm to (47.0, 16.6)
- moved R13 5.00 mm to (59.7, 16.6)
- moved R14 5.00 mm to (63.5, 16.6)
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Connections:
- net A0 renamed IO1
- net A1 renamed IO2
- net A2 renamed IO3
- net A3 renamed IO4
- net A4 renamed IO5
- net A5 renamed IO6
- net A6 renamed IO7
- net A7 renamed IO8
Routing:
- net VIN: track 130.3 -> 227.5 mm
- net IOREF: track 129.8 -> 141.8 mm
- net IO5: track 33.1 -> 25.9 mm
- net IO6: track 44.5 -> 38.2 mm
- net IO4: track 15.5 -> 9.44 mm
- net IO7: track 62.1 -> 57.0 mm
- net IO8: track 73.5 -> 69.6 mm
- net IO3: track 23.7 -> 24.3 mm
Other:
- board size 133.3 x 48.3 mm -> 133 x 40 mm
- board text added: "(c) 2017 SuperHouse Automation Pty Ltd"
- board text added: "1"
- board text added: "2"
- board text added: "3"
- board text added: "4"
- board text added: "5"
- board text added: "6"
- board text added: "7"
- board text added: "8"
- board text added: "GND"
- board text added: "IOREF"
- board text added: "RESET"
- board text added: "SENSOR 1"
- board text added: "SENSOR 2"
- board text added: "SENSOR 3"
- board text added: "SENSOR 4"
- board text added: "SENSOR 5"
- board text added: "SENSOR 6"
- board text added: "SENSOR 7"
- board text added: "SENSOR 8"
- board text added: "SuperHouse"
- board text added: "VIN"
- board text added: "v2.0"
- board text removed: "(c) 2013 Freetronics Pty Ltd"
- board text removed: "12V"
- board text removed: "A0/D0"
- board text removed: "A: A0/D4 B: A1/D5 C: A2/D6 D: A3/D7"
- board text removed: "POWER"
- board text removed: "SENSOR A"
- board text removed: "SENSOR B"
- board text removed: "SENSOR C"
- board text removed: "SENSOR D"
- board text removed: "SENSOR E"
- board text removed: "SENSOR F"
- board text removed: "SENSOR G"
- board text removed: "SENSOR H"
- board text removed: "SUPPLY"
- board text removed: "v1.0"
